File: circular/BOTTOM_pcb_redonda_definitiva.brd (EAGLE design)
At the start: 65 x 65 mm, 9 parts, among them X1 DSB18b20

Commit message: Add files via upload
Parts:
- removed CONECTOR_PLACAS: (no value), pinhead:2X06
- removed EXTRA, EXTRA2: (no value), pinhead:2X10
- removed SD: (no value), pinhead:1X06
- removed X1: DSB18b20, con-wago-500:W237-103
- added 2, C1: JST-XH-06-PIN-LONG-PAD, Rembrandt Electronics - JST XH Connectors v1-0:JST-XH-06-PACKAGE-LONG-PAD
- added B+/B-: (no value), pinhead:2X02
- added DS18B20: JST-XH-03-PIN-LONG-PAD, Rembrandt Electronics - JST XH Connectors v1-0:JST-XH-03-PACKAGE-LONG-PAD
- added SD_MODULE: (no value), pinhead:2X08
- ESPCAM: value (none) -> JST-XH-02-PIN-LONG-PAD; device pinhead:1X03 -> Rembrandt Electronics - JST XH Connectors v1-0:JST-XH-02-PACKAGE-LONG-PAD
- moved ESPCAM 15.0 mm to (57.0, 41.0), flipped to the bottom, turned to 90 degrees
- moved R1 1.00 mm to (18.0, 44.0)
Connections:
- removed net N$7: APC220.1, CONECTOR_PLACAS.2, ESPCAM.1, GY-91.3, R1.1, SD.6, X1.1
- new net N$12: C1.1, SD_MODULE.10, SD_MODULE.9
- new net N$13: SD_MODULE.11, SD_MODULE.12
- new net N$14: 2.1, APC220.1, DS18B20.1, ESPCAM.2, GY-91.3, R1.1, SD_MODULE.13, SD_MODULE.14
- net N$1: now also B+/B-.1, B+/B-.3, C1.5; no longer APC220.2, CONECTOR_PLACAS.4, ESPCAM.3, GY-91.2, SD.5, X1.3
- net N$10: now also C1.2, SD_MODULE.5, SD_MODULE.6; no longer CONECTOR_PLACAS.1, SD.3
- net N$11: now also C1.4, SD_MODULE.7, SD_MODULE.8; no longer CONECTOR_PLACAS.3, SD.4
- net N$2: now also 2.2, APC220.2, B+/B-.2, B+/B-.4, DS18B20.3, ESPCAM.1, GY-91.2, SD_MODULE.1, SD_MODULE.15, SD_MODULE.16, SD_MODULE.2; no longer CONECTOR_PLACAS.7, SD.1
- net N$3: now also 2.5; no longer CONECTOR_PLACAS.10
- net N$4: now also 2.6; no longer CONECTOR_PLACAS.12
- net N$5: now also 2.3; no longer CONECTOR_PLACAS.6
- net N$6: now also 2.4; no longer CONECTOR_PLACAS.8
- net N$8: now also C1.6, DS18B20.2; no longer CONECTOR_PLACAS.11, X1.2
- net N$9: now also C1.3, SD_MODULE.3, SD_MODULE.4; no longer CONECTOR_PLACAS.5, SD.2
Routing:
- net N$14: track 0.00 -> 127.5 mm
- net N$2: track 19.1 -> 134.1 mm
- net N$7: track 106.5 -> 0.00 mm
- net N$1: track 101.9 -> 7.41 mm
- net N$12: track 0.00 -> 21.1 mm
- net N$6: track 31.5 -> 49.3 mm, vias 1 -> 0
- net N$8: track 59.0 -> 42.0 mm
- net N$11: track 15.9 -> 28.4 mm
- net N$9: track 18.3 -> 30.8 mm
- net N$5: track 32.3 -> 42.9 mm
- net N$3: track 42.2 -> 51.8 mm
- net N$4: track 43.2 -> 51.8 mm
- net N$10: track 21.8 -> 27.2 mm
- net N$13: track 0.00 -> 2.58 mm
Other:
- board text added: "BOTTOM"
- board text added: "CANNED UNIVERSE v2.0"
