File: circular/BOTTOM_pcb_redonda_definitiva.sch (EAGLE design)
At the start: 9 parts

Commit message: Add files via upload
Parts:
- removed CONECTOR_PLACAS: (no value), pinhead:PINHD-2X6
- removed EXTRA, JP2: (no value), pinhead:PINHD-2X10
- removed SD: (no value), pinhead:PINHD-1X6
- removed X1: (no value), con-wago-500:W237-103
- added 2, C1: JST-XH-06-PIN-LONG-PAD, Rembrandt Electronics - JST XH Connectors v1-0:JST-XH-06-PIN-LONG-PAD
- added B+/B-: (no value), pinhead:PINHD-2X2
- added DS18B20: JST-XH-03-PIN-LONG-PAD, Rembrandt Electronics - JST XH Connectors v1-0:JST-XH-03-PIN-LONG-PAD
- added SD_MODULE: (no value), pinhead:PINHD-2X8
- ESPCAM: value (none) -> JST-XH-02-PIN-LONG-PAD; device pinhead:PINHD-1X3 -> Rembrandt Electronics - JST XH Connectors v1-0:JST-XH-02-PIN-LONG-PAD
- renumbered T+P+ACC+GY to GY-91
Connections:
- removed net N$7: APC220.1, CONECTOR_PLACAS.2, ESPCAM.1, GY-91.3, R1.1, SD.6, X1-1.KL
- new net N$12: C1-1.S, SD_MODULE.10, SD_MODULE.9
- new net N$13: SD_MODULE.11, SD_MODULE.12
- new net N$14: 2-1.S, APC220.1, DS18B20-1.S, ESPCAM-2.S, GY-91.3, R1.1, SD_MODULE.13, SD_MODULE.14
- net N$1: now also B+/B-.1, B+/B-.3, C1-5.S; no longer APC220.2, CONECTOR_PLACAS.4, ESPCAM.3, GY-91.2, SD.5, X1-3.KL
- net N$10: now also C1-2.S, SD_MODULE.5, SD_MODULE.6; no longer CONECTOR_PLACAS.1, SD.3
- net N$11: now also C1-4.S, SD_MODULE.7, SD_MODULE.8; no longer CONECTOR_PLACAS.3, SD.4
- net N$2: now also 2-2.S, APC220.2, B+/B-.2, B+/B-.4, DS18B20-3.S, ESPCAM-1.S, GY-91.2, SD_MODULE.1, SD_MODULE.15, SD_MODULE.16, SD_MODULE.2; no longer CONECTOR_PLACAS.7, SD.1
- net N$3: now also 2-5.S; no longer CONECTOR_PLACAS.10
- net N$4: now also 2-6.S; no longer CONECTOR_PLACAS.12
- net N$5: now also 2-3.S; no longer CONECTOR_PLACAS.6
- net N$6: now also 2-4.S; no longer CONECTOR_PLACAS.8
- net N$8: now also C1-6.S, DS18B20-2.S; no longer CONECTOR_PLACAS.11, X1-2.KL
- net N$9: now also C1-3.S, SD_MODULE.3, SD_MODULE.4; no longer CONECTOR_PLACAS.5, SD.2
