File: circular/TOP_pcb_redonda_definitiva.sch (EAGLE design)
At the start: 9 parts

Commit message: Add files via upload
Parts:
- removed APC220: (no value), pinhead:PINHD-1X7
- removed CONECTOR_PLACAS: (no value), pinhead:PINHD-2X6
- removed ESPCAM: (no value), pinhead:PINHD-1X3
- removed EXTRA, JP2: (no value), pinhead:PINHD-2X10
- removed SD: (no value), pinhead:PINHD-1X6
- removed T+P+ACC+GY: (no value), pinhead:PINHD-1X8
- added BUZZ: (no value), pinhead:PINHD-1X3
- added GPS: U-BLOX-NEO6V2, u-blox neo-6m v2:U-BLOX-NEO6V2
- added LED: JST-XH-02-PIN-LONG-PAD, Rembrandt Electronics - JST XH Connectors v1-0:JST-XH-02-PIN-LONG-PAD
- added OLED: (no value), pinhead:PINHD-1X4
- added PLACA: ESP32DEVKITV1, ESP32-DEVKITV1:ESP32DEVKITV1
- added X2: JST-XH-06-PIN-LONG-PAD, Rembrandt Electronics - JST XH Connectors v1-0:JST-XH-06-PIN-LONG-PAD
- X1: value (none) -> JST-XH-06-PIN-LONG-PAD; device con-wago-500:W237-103 -> Rembrandt Electronics - JST XH Connectors v1-0:JST-XH-06-PIN-LONG-PAD
Connections:
- new net GPS: BUZZ.3, GPS.GND, OLED.1, PLACA.GND@2
- new net N$12: LED-1.S, R1.1
- new net N$13: BUZZ.1, PLACA.IO27
- new net N$14: PLACA.IO23, X1-1.S
- new net N$15: PLACA.IO19, X1-2.S
- new net N$16: PLACA.IO18, X1-3.S
- new net N$17: PLACA.IO5, X1-4.S
- net N$1: now also BUZZ.2, GPS.VCC, OLED.2, PLACA.3V3, X2-2.S; no longer APC220.2, CONECTOR_PLACAS.4, ESPCAM.3, SD.5, T+P+ACC+GY.2, X1-3.KL
- net N$10: now also PLACA.IO25, X1-6.S; no longer CONECTOR_PLACAS.1, SD.3
- net N$11: now also LED-2.S, PLACA.IO26; no longer CONECTOR_PLACAS.3, SD.4
- net N$2: now also PLACA.GND@1, R1.2, X2-1.S; no longer CONECTOR_PLACAS.7, SD.1
- net N$3: now also PLACA.VIN, X1-5.S; no longer APC220.4, CONECTOR_PLACAS.10
- net N$4: now also OLED.3, PLACA.IO22, X2-3.S; no longer APC220.5, CONECTOR_PLACAS.12
- net N$5: now also OLED.4, PLACA.IO21, X2-4.S; no longer CONECTOR_PLACAS.6, T+P+ACC+GY.4
- net N$6: now also PLACA.IO3, X2-5.S; no longer CONECTOR_PLACAS.8, T+P+ACC+GY.5
- net N$7: now also PLACA.IO1, X2-6.S; no longer APC220.1, CONECTOR_PLACAS.2, ESPCAM.1, R1.1, SD.6, T+P+ACC+GY.3, X1-1.KL
- net N$8: now also GPS.RX, PLACA.IO16; no longer CONECTOR_PLACAS.11, R1.2, X1-2.KL
- net N$9: now also GPS.TX, PLACA.IO17; no longer CONECTOR_PLACAS.5, SD.2
Other:
- moved on the sheet: R1, X1-1, X1-2, X1-3
